Commit message: added robot state publisher, modified urdf

File: src/robot_description/description/building_robot.xacro (robot description, xacro)
@@ -2,6 +2,6 @@
 <robot name="new_car" xmlns:xacro="http://ros.org/wiki/xacro">
   <!-- Define robot constants -->
+  <xacro:property name="base_length" value="1.65"/>
   <xacro:property name="base_width" value="0.92"/>
-  <xacro:property name="base_length" value="1.65"/>
   <xacro:property name="base_height" value="1.13"/>
   <xacro:property name="wheel_radius" value="0.2"/>
@@ -117,3 +117,5 @@
     <origin xyz ="0 0 1.0414" rpy="0 0 0"/>
   </joint>
+  <!-- Gazebo Plugins -->
+  <!-- <xacro: include filename = "robot_description/urdf/gazebo_control.xacro" /> -->
 </robot>
