Commit message: gazebo, rviz, teleop_twist_keyboard launch

File: src/robot_description/description/building_robot.urdf.xacro (robot description, xacro)
@@ -4,6 +4,31 @@
 <!-- |    EDITING THIS FILE BY HAND IS NOT RECOMMENDED                                 | -->
 <!-- =================================================================================== -->
-<robot name="new_car" xmlns:xacro="http://ros.org/wiki/xacro">
+  <robot name="new_car" xmlns:xacro="http://ros.org/wiki/xacro">
   <xacro:include filename="inertia_macros.xacro"/>
+  <xacro:include filename="ros2_control_ackerman.xacro"/>
+  <!-- <xacro:include filename="gazebo_control.xacro"/> -->
+  <!-- Colors -->
+  <material name="White">
+    <color rgba="1.0 1.0 1.0 1.0"/>
+  </material>
+  <material name="Blue">
+      <color rgba="0.0 0.0 1.0 1.0"/>
+  </material>
+  <material name="Gray">
+    <color rgba="0.5 0.5 0.5 1.0"/>
+  </material>
+  <material name="Black">
+      <color rgba="0.1 0.1 0.1 1"/>
+  </material>
+  <material name="Cyan">
+    <color rgba="0 1.0 1.0 1.0"/>
+  </material>
+  <!-- Dummy Root Link
+  <link name="dummy_base_link"/>
+  <joint name="dummy_base_joint" type="fixed">
+    <parent link="dummy_base_link"/>
+    <child link="base_link"/>
+    <origin xyz="0 0 0" rpy="0 0 0"/>
+  </joint> -->
   <!-- Robot Base -->
   <link name="base_link">
@@ -13,7 +38,5 @@
         <mesh filename="package://robot_description/description/meshes/new_car_chassis.stl" scale="0.58 0.58 0.58"/>
       </geometry>
-      <material name="Blue">
-        <color rgba="0.0 0.0 1.0 1"/>
-      </material>
+      <material name="Blue"/>
     </visual>
     <collision>
@@ -41,8 +64,10 @@
         <cylinder length="0.13" radius="0.01"/>
       </geometry>
-      <material name="Gray">
-        <color rgba="0.5 0.5 0.5 1.0"/>
-      </material>
-    </visual>
+      <material name="Black"/>
+    </visual>
+    <!-- added inertia -->
+    <xacro:inertia_cylinder mass="0.001" length="0.13" radius="0.01">
+      <origin rpy="0 0 0" xyz="0 0 0"/>
+    </xacro:inertia_cylinder>
   </link>
   <joint name="Front_Left_steering_joint" type="revolute">
@@ -59,7 +84,5 @@
         <cylinder length="0.13" radius="0.2"/>
       </geometry>
-      <material name="Gray">
-        <color rgba="0.5 0.5 0.5 1.0"/>
-      </material>
+      <material name="Black"/>
     </visual>
     <collision>
@@ -85,8 +108,10 @@
         <cylinder length="0.13" radius="0.01"/>
       </geometry>
-      <material name="Gray">
-        <color rgba="0.5 0.5 0.5 1.0"/>
-      </material>
-    </visual>
+      <material name="Black"/>
+    </visual>
+    <!-- added inertia -->
+    <xacro:inertia_cylinder mass="0.001" length="0.13" radius="0.01">
+      <origin rpy="0 0 0" xyz="0 0 0"/>
+    </xacro:inertia_cylinder>
   </link>
   <joint name="Front_Right_steering_joint" type="revolute">
@@ -103,7 +128,5 @@
         <cylinder length="0.13" radius="0.2"/>
       </geometry>
-      <material name="Gray">
-        <color rgba="0.5 0.5 0.5 1.0"/>
-      </material>
+      <material name="Black"/>
     </visual>
     <collision>
@@ -130,7 +153,5 @@
         <cylinder length="0.17" radius="0.2"/>
       </geometry>
-      <material name="Gray">
-        <color rgba="0.5 0.5 0.5 1.0"/>
-      </material>
+      <material name="Black"/>
     </visual>
     <collision>
@@ -156,7 +177,5 @@
         <cylinder length="0.17" radius="0.2"/>
       </geometry>
-      <material name="Gray">
-        <color rgba="0.5 0.5 0.5 1.0"/>
-      </material>
+      <material name="Black"/>
     </visual>
     <collision>
@@ -183,7 +202,5 @@
         <cylinder length=".0762" radius=".0762"/>
       </geometry>
-      <material name="Cyan">
-        <color rgba="0 1.0 1.0 1.0"/>
-      </material>
+      <material name="Cyan"/>
     </visual>
     <collision>
@@ -202,3 +219,27 @@
     <origin rpy="0 0 0" xyz="0 0 1.0414"/>
   </joint>
+  <!-- Test box
+  <link name="test">
+    <visual>
+      <origin rpy="0 0 0" xyz="0 0 0"/>
+      <geometry>
+        <box size="1.65 0.92 1.13"/>
+      </geometry>
+      <material name="Cyan"/>
+    </visual>
+    <collision>
+      <origin rpy="0 0 0" xyz="0 0 0"/>
+      <geometry>
+        <box size="1.65 0.92 1.13"/>
+      </geometry>
+    </collision>
+    <xacro:inertia_box mass="1.36" x="1.65" y="0.92" z="1.13">
+      <origin rpy="0 0 0" xyz="0 0 0"/>
+    </xacro:inertia_box>
+  </link>
+  <joint name="test_joint" type="fixed">
+    <parent link="base_link"/>
+    <child link="test"/>
+    <origin rpy="0 0 0" xyz="0 0 1.0414"/>
+  </joint> -->
 </robot>

File: src/robot_description/description/gazebo_control.xacro (robot description, xacro)
@@ -1,24 +1,34 @@
-<!-- gazebo_control.xacro-->
 <?xml version="1.0"?>
 <robot xmlns:xacro="http://www.ros.org/wiki/xacro">
+    <!-- <gazebo>
+        <plugin name="gazebo_ros_joint_state_publisher"
+            filename="libgazebo_ros_joint_state_publisher.so">
+            <update_rate>20</update_rate>
+            <joint_name>slider_joint</joint_name>
+            <joint_name>arm_joint</joint_name>
+        </plugin>
+    </gazebo> -->
     <gazebo>
-            <plugin name='ignition::gazebo::systems::AckermannSteering' filename='ignition-gazebo-ackermann-steering-system'>
-                <topic>/cmd_vel</topic>
-                <left_joint>front_left_wheel_joint</left_joint>
-                <left_joint>rear_left_wheel_joint</left_joint>
-                <right_joint>front_right_wheel_joint</right_joint>
-                <right_joint>rear_right_wheel_joint</right_joint>
-                <left_steering_joint>front_left_steering_joint</left_steering_joint>
-                <right_steering_joint>front_right_steering_joint</right_steering_joint>
-                <kingpin_width>0.75</kingpin_width>
-                <steering_limit>0.5</steering_limit>
-                <wheel_base>1.25</wheel_base>
-                <wheel_separation>0.9</wheel_separation>
-                <wheel_radius>0.2</wheel_radius>
-                <min_velocity>-10</min_velocity>
-                <max_velocity>100</max_velocity>
-                <min_acceleration>-30</min_acceleration>
-                <max_acceleration>30</max_acceleration>
-            </plugin>
+        <plugin filename="ignition-gazebo-ackermann-steering-system"  name=
+        "ignition::gazebo::systems::AckermannSteering">
+            <topic>/cmd_vel</topic>
+            <odom_publish_frequency>10</odom_publish_frequency>
+            <odom_topic>odom</odom_topic>
+            <!-- <left_joint>Front_Left_wheel_joint</left_joint> -->
+            <left_joint>Rear_Left_wheel_joint</left_joint>
+            <!-- <right_joint>Front_Right_wheel_joint</right_joint> -->
+            <right_joint>Rear_Right_wheel_joint</right_joint>
+            <left_steering_joint>Front_Left_steering_joint</left_steering_joint>
+            <right_steering_joint>Front_Right_steering_joint</right_steering_joint>
+            <kingpin_width>0.75</kingpin_width>
+            <steering_limit>0.5</steering_limit>
+            <wheel_base>1.25</wheel_base>
+            <wheel_separation>0.9</wheel_separation>
+            <wheel_radius>0.2</wheel_radius>
+            <min_velocity>-10</min_velocity>
+            <max_velocity>100</max_velocity>
+            <min_acceleration>-30</min_acceleration>
+            <max_acceleration>30</max_acceleration>
+        </plugin>
     </gazebo>
 </robot>

Commit message: linked gazebo & rviz to odom

File: src/robot_description/description/building_robot.urdf.xacro (robot description, xacro)
@@ -241,5 +241,5 @@
     <parent link="base_link"/>
     <child link="test"/>
-    <origin rpy="0 0 0" xyz="0 0 1.0414"/>
+    <origin rpy="0 0 0" xyz="0 0 .43"/>
   </joint> -->
 </robot>

File: src/robot_description/description/inertia_macros.xacro (robot description, xacro)
@@ -3,5 +3,5 @@
     <!-- Specify some standard inertial calculations https://en.wikipedia.org/wiki/List_of_moments_of_inertia -->
     <!-- These make use of xacro's mathematical functionality -->
-    <xacro:macro name="inertia_sphere" params="mass radius *origin">
+    <!-- <xacro:macro name="inertia_sphere" params="mass radius *origin">
         <inertial>
             <xacro:insert_block name="origin"/>
@@ -29,4 +29,18 @@
                     izz="${(1/2) * mass * (radius*radius)}" />
         </inertial>
-    </xacro:macro>
+    </xacro:macro> -->
+  <xacro:macro name="box_inertia" params="m w h d">
+    <inertial>
+      <origin xyz="0 0 0" rpy="${pi/2} 0 ${pi/2}"/>
+      <mass value="${m}"/>
+      <inertia ixx="${(m/12) * (h*h + d*d)}" ixy="0.0" ixz="0.0" iyy="${(m/12) * (w*w + d*d)}" iyz="0.0" izz="${(m/12) * (w*w + h*h)}"/>
+    </inertial>
+  </xacro:macro>
+  <xacro:macro name="cylinder_inertia" params="m r h">
+    <inertial>
+      <origin xyz="0 0 0" rpy="${pi/2} 0 0" />
+      <mass value="${m}"/>
+      <inertia ixx="${(m/12) * (3*r*r + h*h)}" ixy = "0" ixz = "0" iyy="${(m/12) * (3*r*r + h*h)}" iyz = "0" izz="${(m/2) * (r*r)}"/>
+    </inertial>
+  </xacro:macro>
 </robot>

File: src/robot_description/description/new_car_master.urdf.xacro (robot description, xacro)
@@ -1,16 +1,9 @@
 <?xml version="1.0"?>
-<robot xmlns:xacro="http://www.ros.org/wiki/xacro"  name="robot">
-    <!-- <xacro:arg name="use_ros2_control" default="true"/>
-    <xacro:arg name="sim_mode" default="false"/> -->
-    <xacro:include filename="building_robot.xacro" />
-    <!-- <xacro:if value="$(arg use_ros2_control)">
-        <xacro:include filename="ros2_control.xacro" />
-    </xacro:if>
-     <xacro:unless value="$(arg use_ros2_control)">
-        <xacro:include filename="gazebo_control.xacro" />
-    </xacro:unless>
-    <xacro:include filename="lidar.xacro" />
-    <xacro:include filename="camera.xacro" />
-    <xacro:include filename="depth_camera.xacro" />
-    <xacro:include filename="face.xacro" />  -->
+<robot name="my_robot" xmlns:xacro="http://www.ros.org/wiki/xacro">
+  <!-- <xacro:include filename="agv_car.xacro" /> -->
+  <xacro:include filename="new_car.xacro" />
+  <xacro:include filename="ros2_control_ackerman.xacro" />
+  <!-- <xacro:include filename="ros2_control_bicycle.xacro" /> -->
+  <!-- <xacro:include filename="lidar.xacro" />
+  <xacro:include filename="depth_camera.xacro" /> -->
 </robot>

File: src/robot_description/description/ros2_control_ackerman.xacro (robot description, xacro)
@@ -5,27 +5,33 @@
       <plugin>ign_ros2_control/IgnitionSystem</plugin>
     </hardware>
-    <joint name="Rear_Left_wheel_joint">
+    <joint name="rear_left_wheel_joint">
       <command_interface name="velocity" />
       <state_interface name="velocity" />
       <state_interface name="position" />
     </joint>
-    <joint name="Rear_Right_wheel_joint">
+    <joint name="rear_right_wheel_joint">
       <command_interface name="velocity" />
       <state_interface name="velocity" />
       <state_interface name="position" />
     </joint>
-    <joint name="Front_Left_steering_joint">
+    <joint name="left_wheel_steering_joint">
       <command_interface name="position" />
       <state_interface name="position" />
     </joint>
-    <joint name="Front_Right_steering_joint">
+    <joint name="right_wheel_steering_joint">
       <command_interface name="position" />
       <state_interface name="position" />
     </joint>
+    <joint name="front_right_wheel_joint">
+      <state_interface name="position" />
+    </joint>
+    <joint name="front_left_wheel_joint">
+      <state_interface name="position" />
+    </joint>
   </ros2_control>
-    <gazebo>
-        <plugin filename="ign_ros2_control-system" name="ign_ros2_control::IgnitionROS2ControlPlugin">
-        <parameters>$(find robot_description)/config/controllers.yaml</parameters>
-        </plugin>
-    </gazebo>
+  <gazebo>
+      <plugin filename="ign_ros2_control-system" name="ign_ros2_control::IgnitionROS2ControlPlugin">
+      <parameters>$(find robot_description)/config/controllers.yaml</parameters>
+      </plugin>
+  </gazebo>
 </robot>
