Commit message: modified urdf to match new car

File: src/robot_description/description/inertia_macros.xacro (robot description, xacro)
@@ -3,31 +3,31 @@
     <!-- Specify some standard inertial calculations https://en.wikipedia.org/wiki/List_of_moments_of_inertia -->
     <!-- These make use of xacro's mathematical functionality -->
-    <!-- <xacro:macro name="inertia_sphere" params="mass radius *origin">
-        <inertial>
-            <xacro:insert_block name="origin"/>
-            <mass value="${mass}" />
-            <inertia ixx="${(2/5) * mass * (radius*radius)}" ixy="0.0" ixz="0.0"
-                    iyy="${(2/5) * mass * (radius*radius)}" iyz="0.0"
-                    izz="${(2/5) * mass * (radius*radius)}" />
-        </inertial>
-    </xacro:macro>
-    <xacro:macro name="inertia_box" params="mass x y z *origin">
-        <inertial>
-            <xacro:insert_block name="origin"/>
-            <mass value="${mass}" />
-            <inertia ixx="${(1/12) * mass * (y*y+z*z)}" ixy="0.0" ixz="0.0"
-                    iyy="${(1/12) * mass * (x*x+z*z)}" iyz="0.0"
-                    izz="${(1/12) * mass * (x*x+y*y)}" />
-        </inertial>
-    </xacro:macro>
-    <xacro:macro name="inertia_cylinder" params="mass length radius *origin">
-        <inertial>
-            <xacro:insert_block name="origin"/>
-            <mass value="${mass}" />
-            <inertia ixx="${(1/12) * mass * (3*radius*radius + length*length)}" ixy="0.0" ixz="0.0"
-                    iyy="${(1/12) * mass * (3*radius*radius + length*length)}" iyz="0.0"
-                    izz="${(1/2) * mass * (radius*radius)}" />
-        </inertial>
-    </xacro:macro> -->
+  <xacro:macro name="inertia_sphere" params="mass radius *origin">
+      <inertial>
+          <xacro:insert_block name="origin"/>
+          <mass value="${mass}" />
+          <inertia ixx="${(2/5) * mass * (radius*radius)}" ixy="0.0" ixz="0.0"
+                  iyy="${(2/5) * mass * (radius*radius)}" iyz="0.0"
+                  izz="${(2/5) * mass * (radius*radius)}" />
+      </inertial>
+  </xacro:macro>
+  <xacro:macro name="inertia_box" params="mass x y z *origin">
+      <inertial>
+          <xacro:insert_block name="origin"/>
+          <mass value="${mass}" />
+          <inertia ixx="${(1/12) * mass * (y*y+z*z)}" ixy="0.0" ixz="0.0"
+                  iyy="${(1/12) * mass * (x*x+z*z)}" iyz="0.0"
+                  izz="${(1/12) * mass * (x*x+y*y)}" />
+      </inertial>
+  </xacro:macro>
+  <xacro:macro name="inertia_cylinder" params="mass length radius *origin">
+      <inertial>
+          <xacro:insert_block name="origin"/>
+          <mass value="${mass}" />
+          <inertia ixx="${(1/12) * mass * (3*radius*radius + length*length)}" ixy="0.0" ixz="0.0"
+                  iyy="${(1/12) * mass * (3*radius*radius + length*length)}" iyz="0.0"
+                  izz="${(1/2) * mass * (radius*radius)}" />
+      </inertial>
+  </xacro:macro>
   <xacro:macro name="box_inertia" params="m w h d">
     <inertial>

File: src/robot_description/description/new_car.xacro (robot description, xacro)
@@ -4,48 +4,47 @@
     <xacro:property name="base_length" value="1.892"/>
     <xacro:property name="base_height" value="0.626"/>
-    <xacro:property name="wheel_radius" value="0.191"/>
-    <xacro:property name="wheel_width" value="0.121"/>
-    <xacro:property name="wheel_ygap" value="-0.06"/>
-    <xacro:property name="wheel_zoff" value="0.123"/>
-    <xacro:property name="wheel_xoff" value="0.756"/>
-    <material name="Black">
-    <color rgba="0 0 0 1" />
-    </material>
-    <material name="Grey">
-        <color rgba="0.8 0.8 0.8 1" />
-    </material>
-    <material name="Orange">
-        <color rgba="1 0.6 0 1" />
-    </material>
-    <material name="White">
-        <color rgba="1 1 1 1" />
-    </material>
+    <xacro:property name="front_wheel_radius" value="0.2"/>
+    <xacro:property name="front_wheel_width" value="0.13"/>
+    <xacro:property name="rear_wheel_radius" value="0.2"/>
+    <xacro:property name="rear_wheel_width" value="0.17"/>
+    <xacro:include filename="inertia_macros.xacro"/>
+  <!-- Colors -->
+  <material name="White">
+    <color rgba="1.0 1.0 1.0 1.0"/>
+  </material>
+  <material name="Blue">
+      <color rgba="0.0 0.0 1.0 1.0"/>
+  </material>
+  <material name="Gray">
+    <color rgba="0.5 0.5 0.5 1.0"/>
+  </material>
+  <material name="Black">
+      <color rgba="0.1 0.1 0.1 1"/>
+  </material>
+  <material name="Cyan">
+    <color rgba="0 1.0 1.0 1.0"/>
+  </material>
     <link name="base_link" />
     <!-- Chassis -->
     <link name="chassis">
         <visual>
-        <origin xyz=".946 .521 -0.313" rpy="0 0 ${pi}" />
-         <geometry>
-                <mesh filename="package://robot_description/description/meshes/agv_chassis.stl"/>
+        <origin xyz="0 -0.01 0" rpy="0 0 0" />
+            <geometry>
+                <mesh filename="package://robot_description/description/meshes/new_car_chassis.stl" scale="0.58 0.58 0.58"/>
             </geometry>
-            <material name="Cyan">
-                <color rgba="0 1.0 1.0 1.0"/>
-            </material>
+            <material name="Blue"/>
         </visual>
         <collision>
-            <origin xyz=".946 .521 -0.313" rpy="0 0 ${pi}" />
+            <origin xyz="0 -0.01 0" rpy="0 0 0" />
                 <geometry>
-                    <mesh filename="package://robot_description/description/meshes/agv_chassis.stl"/>
+                    <mesh filename="package://robot_description/description/meshes/new_car_chassis.stl" scale="0.58 0.58 0.58"/>
                 </geometry>
         </collision>
-        <!-- <xacro:box_inertia m="15" w="${base_width}" d="${base_length}" h="${base_height}"/> -->
-        <inertial>
-        <origin xyz="0 0 0" rpy="0 0 0" />
-        <mass value="100" />
-        <inertia ixx="10.4" ixy="0.0" ixz="0.0" iyy="35.4" iyz="0.0" izz="41.66" />
-        </inertial>
+        <xacro:inertia_box mass="113.4" x="1.65" y="0.92" z="1.13">
+            <origin rpy="0 -0.01 0" xyz="0 0 0"/>
+        </xacro:inertia_box>
     </link>
     <joint name="chassis_joint" type="fixed">
-        <origin xyz="0.8 0 0.5" rpy="0 0 0" />
+        <origin xyz="0 0 0.2" rpy="0 0 0" />
         <parent link="base_link" />
         <child link="chassis" />
@@ -55,22 +54,19 @@
         <visual>
             <geometry>
-                <cylinder radius="${wheel_radius}" length="${wheel_width}"/>
+                <cylinder radius="${rear_wheel_radius}" length="${rear_wheel_width}"/>
             </geometry>
-            <material name="Gray">
-                <color rgba="0.5 0.5 0.5 1.0"/>
-            </material>
+            <material name="Black"/>
         </visual>
-            <collision>
-                <geometry>
-                    <cylinder radius="${wheel_radius}" length="${wheel_width}"/>
-                </geometry>
-            </collision>
-        <inertial>
-        <mass value="11.3" />
-        <inertia ixx="0.26" ixy="0.0" ixz="0.0" iyy="0.26" iyz="0.0" izz="0.51" />
-        </inertial>
+        <collision>
+            <geometry>
+                <cylinder radius="${rear_wheel_radius}" length="${rear_wheel_width}"/>
+            </geometry>
+        </collision>
+        <xacro:inertia_cylinder mass="6.8" length="0.17" radius="0.2">
+            <origin xyz="-0.6 0.42 0" rpy="-1.57 0 0"/>
+        </xacro:inertia_cylinder>
     </link>
     <joint name="rear_left_wheel_joint" type="continuous">
-        <origin xyz="-0.8 0.5 -0.2" rpy="-1.57 0 0" />
+        <origin xyz="-0.6 0.42 0" rpy="-1.57 0 0"/>
         <parent link="chassis" />
         <child link="rear_left_wheel" />
@@ -82,22 +78,19 @@
         <visual>
             <geometry>
-                <cylinder radius="${wheel_radius}" length="${wheel_width}"/>
+                <cylinder radius="${rear_wheel_radius}" length="${rear_wheel_width}"/>
             </geometry>
-            <material name="Gray">
-                <color rgba="0.5 0.5 0.5 1.0"/>
-            </material>
+            <material name="Black"/>
         </visual>
-            <collision>
-                <geometry>
-                    <cylinder radius="${wheel_radius}" length="${wheel_width}"/>
-                </geometry>
-            </collision>
-        <inertial>
-        <mass value="11.3" />
-        <inertia ixx="0.26" ixy="0.0" ixz="0.0" iyy="0.26" iyz="0.0" izz="0.51" />
-        </inertial>
+        <collision>
+            <geometry>
+                <cylinder radius="${rear_wheel_radius}" length="${rear_wheel_width}"/>
+            </geometry>
+        </collision>
+        <xacro:inertia_cylinder mass="6.8" length="0.17" radius="0.2">
+            <origin xyz="-0.6 -0.42 0" rpy="-1.57 0 0" />
+        </xacro:inertia_cylinder>
     </link>
     <joint name="rear_right_wheel_joint" type="continuous">
-        <origin xyz="-0.8 -0.5 -0.2" rpy="-1.57 0 0" />
+        <origin xyz="-0.6 -0.42 0" rpy="-1.57 0 0" />
         <parent link="chassis" />
         <child link="rear_right_wheel" />
@@ -108,10 +101,10 @@
     <link name="left_wheel_steering">
         <inertial>
-        <mass value="0.1"/>
-        <inertia ixx="0" ixy="0.0" ixz="0.0" iyy="0.0" iyz="0.0" izz="0.0" />
+            <mass value="0.1"/>
+            <inertia ixx="0" ixy="0.0" ixz="0.0" iyy="0.0" iyz="0.0" izz="0.0" />
         </inertial>
     </link>
     <joint name="left_wheel_steering_joint" type="revolute">
-        <origin xyz="0.9 0.5 -0.2" rpy="1.57 0 0" />
+        <origin xyz="0.6 0.45 0" rpy="1.57 0 0"/>
         <parent link="chassis" />
         <child link="left_wheel_steering" />
@@ -123,10 +116,10 @@
     <link name="right_wheel_steering">
         <inertial>
-        <mass value="0.1"/>
-        <inertia ixx="0" ixy="0.0" ixz="0.0" iyy="0.0" iyz="0.0" izz="0.0" />
+            <mass value="0.1"/>
+            <inertia ixx="0" ixy="0.0" ixz="0.0" iyy="0.0" iyz="0.0" izz="0.0" />
         </inertial>
     </link>
     <joint name="right_wheel_steering_joint" type="revolute">
-        <origin xyz="0.9 -0.5 -0.2" rpy="1.57 0 0" />
+        <origin xyz="0.6 -0.45 0" rpy="1.57 0 0"/>
         <parent link="chassis" />
         <child link="right_wheel_steering" />
@@ -139,19 +132,16 @@
          <visual>
             <geometry>
-                <cylinder radius="${wheel_radius}" length="${wheel_width}"/>
+                <cylinder radius="${front_wheel_radius}" length="${front_wheel_width}"/>
             </geometry>
-            <material name="Gray">
-                <color rgba="0.5 0.5 0.5 1.0"/>
-            </material>
+            <material name="Black"/>
         </visual>
-            <collision>
-                <geometry>
-                    <cylinder radius="${wheel_radius}" length="${wheel_width}"/>
-                </geometry>
-            </collision>
-        <inertial>
-        <mass value="11.3" />
-        <inertia ixx="0.26" ixy="0.0" ixz="0.0" iyy="0.26" iyz="0.0" izz="0.51" />
-        </inertial>
+        <collision>
+            <geometry>
+                <cylinder radius="${front_wheel_radius}" length="${front_wheel_width}"/>
+            </geometry>
+        </collision>
+        <xacro:inertia_cylinder mass="4.5" length="0.13" radius="0.2">
+            <origin xyz="0.6 0.45 0" rpy="1.57 0 0"/>
+        </xacro:inertia_cylinder>
     </link>
     <joint name="front_left_wheel_joint" type="continuous">
@@ -166,19 +156,16 @@
         <visual>
             <geometry>
-                <cylinder radius="${wheel_radius}" length="${wheel_width}"/>
+                <cylinder radius="${front_wheel_radius}" length="${front_wheel_width}"/>
             </geometry>
-            <material name="Gray">
-                <color rgba="0.5 0.5 0.5 1.0"/>
-            </material>
+            <material name="Black"/>
         </visual>
-            <collision>
-                <geometry>
-                    <cylinder radius="${wheel_radius}" length="${wheel_width}"/>
-                </geometry>
-            </collision>
-        <inertial>
-        <mass value="11.3" />
-        <inertia ixx="0.26" ixy="0.0" ixz="0.0" iyy="0.26" iyz="0.0" izz="0.51" />
-        </inertial>
+        <collision>
+            <geometry>
+                <cylinder radius="${front_wheel_radius}" length="${front_wheel_width}"/>
+            </geometry>
+        </collision>
+        <xacro:inertia_cylinder mass="4.5" length="0.13" radius="0.2">
+            <origin xyz="0.6 -0.45 0" rpy="1.57 0 0"/>
+        </xacro:inertia_cylinder>
     </link>
     <joint name="front_right_wheel_joint" type="continuous">
