Commit message: adjusted steering angle and torque limits

File: src/robot_description/description/new_car.xacro (robot description, xacro)
@@ -41,5 +41,6 @@
                 </geometry>
         </collision>
-        <xacro:inertia_box mass="113.4" x="1.65" y="0.92" z="1.13">
+        <!-- make box slightly smaller than actual to prevent accidental self collision y=0.92-->
+        <xacro:inertia_box mass="113.4" x="1.65" y="0.87" z="1.13">
             <origin rpy="0 -0.01 0" xyz="0 0 0"/>
         </xacro:inertia_box>
@@ -107,9 +108,10 @@
     <joint name="left_wheel_steering_joint" type="revolute">
         <origin xyz="0.6 0.45 0" rpy="1.57 0 0"/>
-        <parent link="chassis" />
-        <child link="left_wheel_steering" />
-        <axis xyz="0 1 0" />
-        <dynamics damping="0.2" />
-        <limit effort="1000.0" lower="-1.57" upper="1.57" velocity="30"/>
+        <parent link="chassis"/>
+        <child link="left_wheel_steering"/>
+        <axis xyz="0 1 0"/>
+        <dynamics damping="0.2"/>
+        <!-- effort = torque (N/m) Lower/upper = steering angle rad-->
+        <limit effort="500.0" lower="-0.785" upper="0.785" velocity="30"/>
     </joint>
     <!-- right steer Link -->
@@ -122,9 +124,10 @@
     <joint name="right_wheel_steering_joint" type="revolute">
         <origin xyz="0.6 -0.45 0" rpy="1.57 0 0"/>
-        <parent link="chassis" />
-        <child link="right_wheel_steering" />
-        <axis xyz="0 1 0" />
-        <dynamics damping="0.2" />
-        <limit effort="1000.0" lower="-1.57" upper="1.57" velocity="30"/>
+        <parent link="chassis"/>
+        <child link="right_wheel_steering"/>
+        <axis xyz="0 1 0"/>
+        <dynamics damping="0.2"/>
+        <!-- effort = torque (N/m) Lower/upper = steering angle rad-->
+        <limit effort="500.0" lower="-0.785" upper="0.785" velocity="30"/>
     </joint>
     <!-- front left wheel Link -->

Commit message: removed collision of steering wheel to chassis

File: src/robot_description/description/new_car.xacro (robot description, xacro)
@@ -36,11 +36,11 @@
         </visual>
         <collision>
-            <origin xyz="0 -0.01 0" rpy="0 0 0" />
+            <!-- <origin xyz="0 -0.01 0" rpy="0 0 0" />
                 <geometry>
                     <mesh filename="package://robot_description/description/meshes/new_car_chassis.stl" scale="0.58 0.58 0.58"/>
-                </geometry>
+                </geometry> -->
         </collision>
         <!-- make box slightly smaller than actual to prevent accidental self collision y=0.92-->
-        <xacro:inertia_box mass="113.4" x="1.65" y="0.87" z="1.13">
+        <xacro:inertia_box mass="150" x="1.65" y="0.92" z="1.13">
             <origin rpy="0 -0.01 0" xyz="0 0 0"/>
         </xacro:inertia_box>
@@ -113,5 +113,5 @@
         <dynamics damping="0.2"/>
         <!-- effort = torque (N/m) Lower/upper = steering angle rad-->
-        <limit effort="500.0" lower="-0.785" upper="0.785" velocity="30"/>
+        <limit effort="100.0" lower="-0.785" upper="0.785" velocity="30"/>
     </joint>
     <!-- right steer Link -->
@@ -129,5 +129,5 @@
         <dynamics damping="0.2"/>
         <!-- effort = torque (N/m) Lower/upper = steering angle rad-->
-        <limit effort="500.0" lower="-0.785" upper="0.785" velocity="30"/>
+        <limit effort="100.0" lower="-0.785" upper="0.785" velocity="30"/>
     </joint>
     <!-- front left wheel Link -->

Commit message: added lidar, ros gz bridge

File: src/robot_description/description/new_car.xacro (robot description, xacro)
@@ -9,20 +9,23 @@
     <xacro:property name="rear_wheel_width" value="0.17"/>
     <xacro:include filename="inertia_macros.xacro"/>
-  <!-- Colors -->
-  <material name="White">
-    <color rgba="1.0 1.0 1.0 1.0"/>
-  </material>
-  <material name="Blue">
-      <color rgba="0.0 0.0 1.0 1.0"/>
-  </material>
-  <material name="Gray">
-    <color rgba="0.5 0.5 0.5 1.0"/>
-  </material>
-  <material name="Black">
-      <color rgba="0.1 0.1 0.1 1"/>
-  </material>
-  <material name="Cyan">
-    <color rgba="0 1.0 1.0 1.0"/>
-  </material>
+    <!-- Colors -->
+    <material name="White">
+        <color rgba="1.0 1.0 1.0 1.0"/>
+    </material>
+    <material name="Blue">
+        <color rgba="0.0 0.0 1.0 1.0"/>
+    </material>
+    <material name="Gray">
+        <color rgba="0.5 0.5 0.5 1.0"/>
+    </material>
+    <material name="Black">
+        <color rgba="0.1 0.1 0.1 1"/>
+    </material>
+    <material name="Cyan">
+        <color rgba="0 1.0 1.0 1.0"/>
+    </material>
+    <material name="Red">
+        <color rgba="1 0 0 1.0"/>
+    </material>
     <link name="base_link" />
     <!-- Chassis -->
@@ -179,6 +182,6 @@
         <dynamics damping="0.2" />
     </joint>
-        <!-- Lidar -->
-    <link name="velodyne">
+    <!-- Lidar -->
+    <!-- <link name="velodyne">
         <visual>
             <origin xyz="0 0 0" rpy="0 0 0"/>
@@ -186,7 +189,13 @@
                 <cylinder radius=".0762" length=".0762"/>
             </geometry>
-            <material name="Cyan">
-                <color rgba="0 1.0 1.0 1.0"/>
-            </material>
+            <material name="Cyan"/>
+            <collision>
+                <geometry>
+                    <cylinder radius=".0762" length=".0762"/>
+                </geometry>
+            </collision>
+        <xacro:inertia_cylinder mass="2" length=".0762" radius=".0762">
+            <origin xyz="0 0 0" rpy="0 0 0"/>
+        </xacro:inertia_cylinder>
         </visual>
     </link>
@@ -195,4 +204,4 @@
         <child link="velodyne"/>
         <origin xyz="0 0 1.0414" rpy="0 0 0"/>
-    </joint>
+    </joint> -->
 </robot>

File: src/robot_description/description/new_car_master.urdf.xacro (robot description, xacro)
@@ -1,9 +1,8 @@
 <?xml version="1.0"?>
 <robot name="my_robot" xmlns:xacro="http://www.ros.org/wiki/xacro">
-  <!-- <xacro:include filename="agv_car.xacro" /> -->
   <xacro:include filename="new_car.xacro" />
+  <!-- <xacro:include filename="gazebo_control.xacro" /> -->
   <xacro:include filename="ros2_control_ackerman.xacro" />
-  <!-- <xacro:include filename="ros2_control_bicycle.xacro" /> -->
-  <!-- <xacro:include filename="lidar.xacro" />
-  <xacro:include filename="depth_camera.xacro" /> -->
+  <xacro:include filename="lidar.xacro" />
+  <!-- <xacro:include filename="depth_camera.xacro" /> -->
 </robot>
