Commit message: added depth camera

File: src/robot_description/description/gazebo_control.xacro (robot description, xacro)
@@ -1,13 +1,13 @@
 <?xml version="1.0"?>
 <robot xmlns:xacro="http://www.ros.org/wiki/xacro">
+    <gazebo reference="front_right_wheel">
+        <mu1 value="0.5"/>
+        <mu2 value="0.5"/>
+    </gazebo>
+    <gazebo reference="front_left_wheel">
+        <mu1 value="0.5"/>
+        <mu2 value="0.5"/>
+    </gazebo>
     <!-- <gazebo>
-        <plugin name="gazebo_ros_joint_state_publisher"
-            filename="libgazebo_ros_joint_state_publisher.so">
-            <update_rate>20</update_rate>
-            <joint_name>slider_joint</joint_name>
-            <joint_name>arm_joint</joint_name>
-        </plugin>
-    </gazebo> -->
-    <gazebo>
         <plugin filename="ignition-gazebo-ackermann-steering-system"  name=
         "ignition::gazebo::systems::AckermannSteering">
@@ -15,7 +15,7 @@
             <odom_publish_frequency>10</odom_publish_frequency>
             <odom_topic>odom</odom_topic>
-            <!-- <left_joint>Front_Left_wheel_joint</left_joint> -->
+             <left_joint>Front_Left_wheel_joint</left_joint>
             <left_joint>Rear_Left_wheel_joint</left_joint>
-            <!-- <right_joint>Front_Right_wheel_joint</right_joint> -->
+            <right_joint>Front_Right_wheel_joint</right_joint>
             <right_joint>Rear_Right_wheel_joint</right_joint>
             <left_steering_joint>Front_Left_steering_joint</left_steering_joint>
@@ -31,4 +31,4 @@
             <max_acceleration>30</max_acceleration>
         </plugin>
-    </gazebo>
+    </gazebo> -->
 </robot>

File: src/robot_description/description/lidar.xacro (robot description, xacro)
@@ -5,5 +5,5 @@
         <parent link="chassis"/>
         <child link="laser_frame"/>
-        <origin xyz="0 0 1.0414" rpy="0 0 0"/>
+        <origin xyz="-0.1 0 1.1" rpy="0 0 0"/>
     </joint>
     <link name="laser_frame">
@@ -12,5 +12,7 @@
                 <cylinder radius="0.05" length="0.05"/>
             </geometry>
-            <material name="purple"/>
+            <material name="Cyan">
+                <color rgba="0 1.0 1.0 1.0"/>
+            </material>
         </visual>
         <collision>
@@ -25,5 +27,4 @@
     <!-- 3D Lidar New Gazebo Sensor Plugin  -->
     <gazebo reference="laser_frame">
-        <material>Gazebo/Purple</material>
         <sensor name="laser" type="gpu_lidar">
             <pose> 0 0 0 0 0 0 </pose>
@@ -42,6 +43,6 @@
                     <vertical>
                         <samples>40</samples>
-                        <min_angle>-0.186</min_angle>
-                        <max_angle>0.186</max_angle>
+                        <min_angle>-0.26</min_angle>
+                        <max_angle>0.26</max_angle>
                     </vertical>
                 </scan>

File: src/robot_description/description/new_car_master.urdf.xacro (robot description, xacro)
@@ -2,7 +2,8 @@
 <robot name="my_robot" xmlns:xacro="http://www.ros.org/wiki/xacro">
   <xacro:include filename="new_car.xacro" />
-  <!-- <xacro:include filename="gazebo_control.xacro" /> -->
   <xacro:include filename="ros2_control_ackerman.xacro" />
   <xacro:include filename="lidar.xacro" />
+  <xacro:include filename="cameras.xacro" />
+  <xacro:include filename="gazebo_control.xacro" />
   <!-- <xacro:include filename="depth_camera.xacro" /> -->
 </robot>

Commit message: added IMU sensors

File: src/robot_description/description/gazebo_control.xacro (robot description, xacro)
@@ -8,4 +8,12 @@
         <mu1 value="0.5"/>
         <mu2 value="0.5"/>
+    </gazebo>
+    <gazebo reference="imu_link">
+        <sensor name="imu_sensor" type="imu">
+            <always_on>1</always_on>
+            <update_rate>1</update_rate>
+            <visualize>true</visualize>
+            <topic>imu</topic>
+        </sensor>
     </gazebo>
     <!-- <gazebo>

File: src/robot_description/description/new_car.xacro (robot description, xacro)
@@ -182,26 +182,18 @@
         <dynamics damping="0.2" />
     </joint>
-    <!-- Lidar -->
-    <!-- <link name="velodyne">
+    <!-- IMU -->
+    <joint name="imu_joint" type="fixed">
+        <origin xyz="0 0 0" rpy="0 0 0" />
+        <parent link="chassis" />
+        <child link="imu_link" />
+    </joint>
+    <link name="imu_link">
+        <pose>0 0 0 0 0 0</pose>  <!-- Adjust height based on your vehicle -->
         <visual>
-            <origin xyz="0 0 0" rpy="0 0 0"/>
             <geometry>
-                <cylinder radius=".0762" length=".0762"/>
+                <box size ="0.05 0.05 0.01"/>
             </geometry>
-            <material name="Cyan"/>
-            <collision>
-                <geometry>
-                    <cylinder radius=".0762" length=".0762"/>
-                </geometry>
-            </collision>
-        <xacro:inertia_cylinder mass="2" length=".0762" radius=".0762">
-            <origin xyz="0 0 0" rpy="0 0 0"/>
-        </xacro:inertia_cylinder>
+            <material name ="White"/>
         </visual>
     </link>
-    <joint name="velodyne_joint" type="fixed">
-        <parent link="chassis"/>
-        <child link="velodyne"/>
-        <origin xyz="0 0 1.0414" rpy="0 0 0"/>
-    </joint> -->
 </robot>
