Commit message: added front, right depth cameras

File: src/robot_description/description/cameras.xacro (robot description, xacro)
@@ -5,7 +5,14 @@
         <parent link="chassis"/>
         <child link="camera_link"/>
-        <origin xyz="0.27 0 1.1" rpy="0 0 0"/>
+        <origin xyz="0 0 0.5" rpy="0 0 0"/>
     </joint>
-    <link name="camera_link">
+    <link name="camera_link"></link>
+    <!-- Front camera Optical link -->
+    <joint name="front_camera_joint" type="fixed">
+        <parent link="camera_link"/>
+        <child link="front_camera"/>
+        <origin xyz="0.5 0 0" rpy="0 0 0"/>
+    </joint>
+    <link name="front_camera">
         <visual>
             <geometry>
@@ -15,25 +22,18 @@
         </visual>
     </link>
-    <!-- Depth camera Optical link -->
-    <joint name="camera_optical_joint" type="fixed">
-        <parent link="camera_link"/>
-        <child link="camera_link_optical"/>
-        <origin xyz="0 0 0" rpy="0 0 0"/>
-    </joint>
-    <link name="camera_link_optical"></link>
-    <!-- Depth camera Gazebo Sensor Plugin -->
-    <gazebo reference="camera_link">
+    <!-- Front camera Gazebo Sensor Plugin -->
+    <gazebo reference="front_camera">
         <material>Gazebo/Black</material>
-        <sensor name="rgbd_camera" type="rgbd_camera">
+        <sensor name="rgbd_camera1" type="rgbd_camera">
             <pose> 0 0 0 0 0 0 </pose>
             <always_on>true</always_on>
             <visualize>true</visualize>
             <update_rate>30</update_rate>
-            <topic>camera</topic>
+            <topic>camera1</topic>
             <gz_frame_id>camera_link</gz_frame_id>
             <camera>
-                <optical_frame_id>camera_link_optical</optical_frame_id>
+                <optical_frame_id>front_camera</optical_frame_id>
                 <camera_info_topic>camera/camera_info</camera_info_topic>
-                <horizontal_fov>1.089</horizontal_fov>
+                <horizontal_fov>1.52</horizontal_fov>
                 <image>
                     <format>R8G8B8</format>
@@ -43,5 +43,45 @@
                 <clip>
                     <near>0.05</near>
-                    <far>8.0</far>
+                    <far>6.0</far>
+                </clip>
+            </camera>
+        </sensor>
+    </gazebo>
+       <!-- Right camera Optical link -->
+    <joint name="right_camera_joint" type="fixed">
+        <parent link="camera_link"/>
+        <child link="right_camera"/>
+        <origin xyz="0 -0.27 0" rpy="0 0 -1.57"/>
+    </joint>
+    <link name="right_camera">
+        <visual>
+            <geometry>
+                <box size="0.04 0.04 0.04"/>
+            </geometry>
+            <material name="black"/>
+        </visual>
+    </link>
+    <!-- Right camera Gazebo Sensor Plugin -->
+    <gazebo reference="right_camera">
+        <material>Gazebo/Black</material>
+        <sensor name="rgbd_camera2" type="rgbd_camera">
+            <pose> 0 0 0 0 0 0 </pose>
+            <always_on>true</always_on>
+            <visualize>true</visualize>
+            <update_rate>30</update_rate>
+            <topic>camera2</topic>
+            <gz_frame_id>camera_link</gz_frame_id>
+            <camera>
+                <optical_frame_id>right_camera</optical_frame_id>
+                <camera_info_topic>camera/camera_info</camera_info_topic>
+                <horizontal_fov>1.52</horizontal_fov>
+                <image>
+                    <format>R8G8B8</format>
+                    <width>640</width>
+                    <height>480</height>
+                </image>
+                <clip>
+                    <near>0.05</near>
+                    <far>6.0</far>
                 </clip>
             </camera>

Commit message: fixed parking detection

File: src/robot_description/description/cameras.xacro (robot description, xacro)
@@ -38,6 +38,6 @@
                 <image>
                     <format>R8G8B8</format>
-                    <width>640</width>
-                    <height>480</height>
+                    <width>600</width>
+                    <height>400</height>
                 </image>
                 <clip>
@@ -78,6 +78,6 @@
                 <image>
                     <format>R8G8B8</format>
-                    <width>640</width>
-                    <height>480</height>
+                    <width>600</width>
+                    <height>400</height>
                 </image>
                 <clip>

File: src/robot_description/description/new_car.xacro (robot description, xacro)
@@ -34,5 +34,5 @@
         <origin xyz="0 -0.01 0" rpy="0 0 0" />
             <geometry>
-                <mesh filename="package://robot_description/description/meshes/new_car_chassis.stl" scale="0.58 0.58 0.58"/>
+                <mesh filename="package://robot_description/description/meshes/new_car_chassis.stl" scale="0.58 0.5 0.58"/>
             </geometry>
             <material name="Blue"/>

File: src/robot_description/description/new_car_master.urdf.xacro (robot description, xacro)
@@ -3,5 +3,5 @@
   <xacro:include filename="new_car.xacro" />
   <xacro:include filename="ros2_control_ackerman.xacro" />
-  <xacro:include filename="lidar.xacro" />
+  <!-- <xacro:include filename="lidar.xacro" /> -->
   <xacro:include filename="cameras.xacro" />
   <xacro:include filename="gazebo_control.xacro" />
